File: ATMEGA32_DEV.sch (EAGLE design)
At the start: 17 parts, among them IC1 MEGA32-A, IC2 7805T, Q1 16MHz

Commit message: Included mounting holes
Parts:
- removed CN2: (no value), adafruit:DCBARRELPTH
- added H1, H2, H3, H4: MOUNT-HOLE2.8, holes:MOUNT-HOLE2.8
- added J1: DCJ0202, con-jack:DCJ0202
Connections:
- net GND: now also J1.2, J1.3; no longer CN2.GND
- net N$3: now also J1.1; no longer CN2.PWR
Changed lines of the file:
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@@
 <part name="JP3" library="adafruit" library_urn="urn:adsk.eagle:library:420" deviceset="PINHD-2X4" device="" package3d_urn="urn:adsk.eagle:package:6240893/1"/>
 <part name="JP4" library="adafruit" library_urn="urn:adsk.eagle:library:420" deviceset="PINHD-2X4" device="" package3d_urn="urn:adsk.eagle:package:6240893/1"/>
-<part name="CN2" library="adafruit" library_urn="urn:adsk.eagle:library:420" deviceset="DCBARREL" device="PTH" package3d_urn="urn:adsk.eagle:package:6240729/1"/>
 <part name="IC2" library="linear" library_urn="urn:adsk.eagle:library:262" deviceset="78*" device="T" package3d_urn="urn:adsk.eagle:package:16414/1" technology="05"/>
 <part name="C3" library="rcl" library_urn="urn:adsk.eagle:library:334" deviceset="C-EU" device="C0805" package3d_urn="urn:adsk.eagle:package:23617/2" value="100uF"/>
@@
 <part name="SW1" library="adafruit" library_urn="urn:adsk.eagle:library:420" deviceset="SWITCH_PUSHBUTTON" device="EVQ-PE" package3d_urn="urn:adsk.eagle:package:6240957/1"/>
 <part name="GND7" library="supply1" library_urn="urn:adsk.eagle:library:371" deviceset="GND" device=""/>
+<part name="H1" library="holes" library_urn="urn:adsk.eagle:library:237" deviceset="MOUNT-HOLE" device="2.8" package3d_urn="urn:adsk.eagle:package:14271/1"/>
+<part name="H2" library="holes" library_urn="urn:adsk.eagle:library:237" deviceset="MOUNT-HOLE" device="2.8" package3d_urn="urn:adsk.eagle:package:14271/1"/>
+<part name="H3" library="holes" library_urn="urn:adsk.eagle:library:237" deviceset="MOUNT-HOLE" device="2.8" package3d_urn="urn:adsk.eagle:package:14271/1"/>
+<part name="H4" library="holes" library_urn="urn:adsk.eagle:library:237" deviceset="MOUNT-HOLE" device="2.8" package3d_urn="urn:adsk.eagle:package:14271/1"/>
+<part name="J1" library="con-jack" library_urn="urn:adsk.eagle:library:154" deviceset="DCJ0202" device="" package3d_urn="urn:adsk.eagle:package:7491/1"/>
 </parts>
 <sheets>
@@
 <attribute name="VALUE" x="1344.93" y="1099.82" size="1.778" layer="96"/>
 </instance>
-<instance part="CN2" gate="G$1" x="1132.84" y="1206.5" smashed="yes">
-<attribute name="NAME" x="1127.76" y="1211.58" size="1.27" layer="95"/>
-<attribute name="VALUE" x="1127.76" y="1201.42" size="1.27" layer="96"/>
-</instance>
 <instance part="IC2" gate="A1" x="1176.02" y="1209.04" smashed="yes">
 <attribute name="NAME" x="1168.4" y="1214.755" size="1.778" layer="95"/>
@@
 <instance part="GND7" gate="1" x="1249.68" y="1198.88" smashed="yes" rot="R90">
 <attribute name="VALUE" x="1252.22" y="1196.34" size="1.778" layer="96" rot="R90"/>
+</instance>
+<instance part="H1" gate="G$1" x="1150.62" y="1150.62" smashed="yes">
+<attribute name="NAME" x="1152.652" y="1151.2042" size="1.778" layer="95"/>
+<attribute name="VALUE" x="1152.652" y="1148.1562" size="1.778" layer="96"/>
+</instance>
+<instance part="H2" gate="G$1" x="1150.62" y="1143" smashed="yes">
+<attribute name="NAME" x="1152.652" y="1143.5842" size="1.778" layer="95"/>
+<attribute name="VALUE" x="1152.652" y="1140.5362" size="1.778" layer="96"/>
+</instance>
+<instance part="H3" gate="G$1" x="1183.64" y="1150.62" smashed="yes">
+<attribute name="NAME" x="1185.672" y="1151.2042" size="1.778" layer="95"/>
+<attribute name="VALUE" x="1185.672" y="1148.1562" size="1.778" layer="96"/>
+</instance>
+<instance part="H4" gate="G$1" x="1183.64" y="1143" smashed="yes">
+<attribute name="NAME" x="1185.672" y="1143.5842" size="1.778" layer="95"/>
+<attribute name="VALUE" x="1185.672" y="1140.5362" size="1.778" layer="96"/>
+</instance>
+<instance part="J1" gate="G$1" x="1127.76" y="1206.5" smashed="yes">
+<attribute name="NAME" x="1125.22" y="1210.31" size="1.778" layer="95"/>
+<attribute name="VALUE" x="1125.22" y="1200.15" size="1.778" layer="96"/>
 </instance>
 </instances>
@@
 <pinref part="C5" gate="G$1" pin="-"/>
 <wire x1="1155.7" y1="1193.8" x2="1143" y2="1193.8" width="0.1524" layer="91"/>
-<pinref part="CN2" gate="G$1" pin="GND"/>
 <wire x1="1143" y1="1193.8" x2="1135.38" y2="1193.8" width="0.1524" layer="91"/>
 <wire x1="1135.38" y1="1193.8" x2="1135.38" y2="1203.96" width="0.1524" layer="91"/>
@@
 <junction x="1203.96" y="1196.34"/>
 <pinref part="GND6" gate="1" pin="GND"/>
+<pinref part="J1" gate="G$1" pin="3"/>
+<pinref part="J1" gate="G$1" pin="2"/>
+<wire x1="1135.38" y1="1206.5" x2="1135.38" y2="1203.96" width="0.1524" layer="91"/>
+<junction x="1135.38" y="1203.96"/>
 </segment>
 <segment>
@@
 <net name="N$3" class="0">
 <segment>
-<pinref part="CN2" gate="G$1" pin="PWR"/>
 <pinref part="C5" gate="G$1" pin="+"/>
 <wire x1="1135.38" y1="1209.04" x2="1143" y2="1209.04" width="0.1524" layer="91"/>
@@
 <wire x1="1155.7" y1="1209.04" x2="1165.86" y2="1209.04" width="0.1524" layer="91"/>
 <junction x="1155.7" y="1209.04"/>
-</segment>
-</net>
+<pinref part="J1" gate="G$1" pin="1"/>
+</segment>
+</net>
