File: ATMEGA32_DEV.brd (EAGLE design)
At the start: 87.6 x 51.7 mm, 17 parts, among them IC1 MEGA32-A, IC2 7805T, Q1 16MHz

Commit message: re_adjusted layout
Parts:
- removed CN2: (no value), adafruit:DCJACK_2MM_PTH
- added H1, H2, H3, H4: MOUNT-HOLE2.8, holes:2,8
- added J1: DCJ0202, con-jack:DCJ0202
- moved C3 10.5 mm to (40.6, 40.6)
- moved C4 10.2 mm to (49.5, 40.6)
- moved IC2 7.62 mm to (44.5, 59.7)
- moved C5 3.59 mm to (31.8, 57.1)
Connections:
- removed net GNDBREAK: CN2.GNDBREAK
- net GND: now also J1.2, J1.3; no longer CN2.GND
- net N$3: now also J1.1; no longer CN2.PWR
Routing:
- net GND: track 249.3 -> 259.0 mm, vias 5 -> 4
- net +5V: track 205.5 -> 214.6 mm
- net N$3: track 39.5 -> 35.7 mm
